File: atslim-328.kicad_pcb (KiCad board)
At the start: 2 copper layers, 65 x 30 mm, 58 parts, among them IC1 SN74LVC125ADRG3, J1 UPDI, J2 RESET, J3 Micro_SD_Card_Det1, J4 USB4500-03-0-A_REVA1, J5 1888250-3, J6 GPIO, U1 ATmega3208-M, U2 LT1963AxST-3.3, U3 W5500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

Commit message: Cleanup and added PoE header
Parts:
- added J7: PoE Header, Connector_PinHeader_2.54mm:PinHeader_2x02_P2.54mm_Vertical, F.Cu at (94.8, 97.5)
- R15, R18: moved to B.Cu
- R20, R21: moved to F.Cu
- moved R21 11.6 mm to (92.6, 79.0)
- moved R20 10.7 mm to (91.7, 94.1)
- moved R19 3.88 mm to (95.2, 80.3), turned to 180 degrees
- moved C10 1.96 mm to (92.6, 80.3), turned to 0 degrees
- moved R14 1.26 mm to (90.9, 87.8)
- moved C8 1.19 mm to (101.2, 88.9)
- moved C9 1.19 mm to (100.5, 88.2)
- moved R13 1.19 mm to (102.0, 89.7)
- moved R15 0.94 mm to (90.9, 88.8), turned to -90 degrees
- moved C11 0.60 mm to (89.2, 88.4)
- moved C12 0.60 mm to (89.2, 86.4)
- moved R22 0.20 mm to (107.0, 77.3)
Connections:
- net /ethernet/RD+ renamed Net-(J5-RD+)
- net /ethernet/RD- renamed Net-(J5-RD-)
- net /ethernet/TD+ renamed /ethernet/TX+
- net /ethernet/TD- renamed /ethernet/TX-
Routing:
- net SPI_MOSI: track 42.5 -> 26.3 mm, vias 5 -> 3
- net TR1_TAP: track 0.00 -> 14.6 mm, vias 0 -> 2
- net TR0_TAP: track 0.00 -> 12.9 mm, vias 0 -> 2
- net /ethernet/LINK_LED: track 31.9 -> 19.7 mm, vias 3 -> 2
- net /ethernet/ACT_LED: track 25.2 -> 13.2 mm, vias 1 -> 0
- net Net-(J5-LED2_DAT): track 5.31 -> 14.9 mm
- net Net-(J5-LED1_DAT): track 3.90 -> 12.9 mm, vias 0 -> 1
- net SPI_SCK: track 37.3 -> 31.8 mm, vias 5 -> 3
- net /ethernet/RX+: track 9.61 -> 14.5 mm
- net Net-(J5-TCT): track 9.41 -> 12.4 mm
- net +3V3: track 151.4 -> 153.4 mm, vias 2 -> 3
- net /ethernet/RX-: track 13.3 -> 11.9 mm, vias 2 -> 1
- net GND: track 43.4 -> 44.6 mm, vias 23 -> 22
- net Net-(R13-Pad2): track 2.10 -> 3.30 mm
- net Net-(U3-TOCAP): track 2.23 -> 3.29 mm
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
Commit message: Sent off to manufacturer for test articles
Parts:
- J7: value PoE Header -> PoE
- moved C3 0.54 mm to (118.9, 81.9)
- moved C6 0.50 mm to (108.7, 92.4)
- moved C4 0.19 mm to (117.8, 80.8)
Routing:
- net CS_LLS: track 7.63 -> 6.32 mm
- net SPI_MISO: track 35.6 -> 34.6 mm, vias 4 -> 3
- net /DIGF5: track 22.0 -> 22.9 mm
- net SPI_MOSI: track 26.3 -> 27.0 mm
- net +3V3: track 153.4 -> 154.1 mm, vias 3 -> 5
- net SPI_SCK: track 31.8 -> 31.2 mm
- net Net-(U1-AVDD): track 5.63 -> 5.07 mm
- net GND: track 44.6 -> 44.1 mm
- net SPI_CS: track 18.3 -> 18.7 mm, vias 4 -> 2
- net +5V: track 57.9 -> 57.8 mm, vias 5 -> 4

Commit message: Recent updates
Parts:
- removed J7: PoE, Connector_PinHeader_2.54mm:PinHeader_2x02_P2.54mm_Vertical
- removed X1: 25MHz, Crystal:Crystal_SMD_TXC_9HT11-2Pin_2.0x1.2mm_HandSoldering
- added P1: PoE Header, Connector_PinHeader_2.54mm:PinHeader_1x02_P2.54mm_Vertical, F.Cu at (93.8, 97.5)
- added Y1: 830081609, CrystalOscillator:830081609, F.Cu at (107.6, 92.7)
- C5, C6: moved to B.Cu
- moved C5 2.61 mm to (107.0, 91.7), turned to 90 degrees
- moved R20 1.42 mm to (93.1, 94.1)
- moved C6 1.38 mm to (108.2, 93.7), turned to -90 degrees
- moved R12 0.40 mm to (105.1, 92.1)
- moved R22 0.19 mm to (106.9, 77.4)
Connections:
- C5 pad 1: Net-(U3-XI/CLKIN) -> Net-(Y1-GND_1)
- C6 pad 1: Net-(U3-XO) -> Net-(Y1-GND_2)
- J5 pad 7: TR0_TAP -> V+
- J5 pad 8: TR1_TAP -> V-
- J6 pad 1: GND -> +3V3
- J6 pad 2: +3V3 -> GND
Routing:
- net V-: track 0.00 -> 16.0 mm
- net V+: track 0.00 -> 15.0 mm
- net TR1_TAP: track 14.6 -> 0.00 mm, vias 2 -> 0
- net TR0_TAP: track 12.9 -> 0.00 mm, vias 2 -> 0
- net +3V3: track 154.1 -> 145.3 mm
- net RESET: track 32.8 -> 28.2 mm
- net Net-(J2-COM_2): track 37.5 -> 34.8 mm
- net GND: track 44.1 -> 41.9 mm, vias 22 -> 21
- net Net-(U3-XI/CLKIN): track 6.45 -> 4.84 mm
- net Net-(J5-LED1_DAT): track 12.9 -> 14.3 mm
- net /ethernet/ACT_LED: track 13.2 -> 11.8 mm
- net Net-(C1-Pad1): track 1.13 -> 0.00 mm
- net CS_LLS: track 6.32 -> 5.67 mm
- net Net-(D1-A): track 2.83 -> 3.47 mm
- net Net-(Y1-GND_2): vias 0 -> 1
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- added copper zone on F.Cu, net +3V3
- added copper zone on F.Cu, net Net-(C1-Pad1)
- added copper zone on F.Cu, net Net-(J2-COM_2)
- added copper zone on F.Cu, net RESET
Other:
- board text added: "PoE"
- board text added: "ZMT"
- board text added: "{ "ViaStitching": "0.2", "stitch_zone_0": { "HSpacing": "1", "VSpacing": "1", "Clearance": "1", "Randomize": false } }"

Commit message: Fucked up UPDI... of course
Connections:
- J1 pad 3: Prog_TX -> unconnected-(J1-NC-Pad3)
- J1 pad 5: unconnected-(J1-Pad5) -> Prog_TX
Routing:
- net Prog_TX: track 22.3 -> 23.6 mm
Changed lines of the file:
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@@
 	(net 82 "/DIGD4")
 	(net 83 "/DIGF5")
-	(net 84 "unconnected-(J1-Pad5)")
+	(net 84 "unconnected-(J1-NC-Pad3)")
 	(net 85 "Prog_RX")
 	(net 86 "/UPDI")
@@
 			(size 0.7874 0.7874)
 			(layers "F.Cu" "F.Mask")
-			(net 87 "Prog_TX")
-			(pinfunction "TX")
-			(pintype "output")
+			(net 84 "unconnected-(J1-NC-Pad3)")
+			(pinfunction "NC")
+			(pintype "open_collector+no_connect")
 		)
 		(pad "4" connect circle
@@
 			(size 0.7874 0.7874)
 			(layers "F.Cu" "F.Mask")
-			(net 84 "unconnected-(J1-Pad5)")
-			(pintype "open_collector+no_connect")
+			(net 87 "Prog_TX")
+			(pinfunction "TX")
+			(pintype "output")
 		)
 		(pad "6" connect circle
@@
 	)
 	(segment
-		(start 106.416765 79.483235)
-		(end 106.133921 79.483235)
-		(width 0.2)
-		(layer "F.Cu")
-		(net 87)
-	)
-	(segment
-		(start 100.585686 73.935)
-		(end 97.43 73.935)
+		(start 96.16 73.935)
+		(end 95.4 74.695)
 		(width 0.2)
 		(layer "F.Cu")
@@
 	)
 	(segment
-		(start 109.115 85.08)
-		(end 110.614455 85.08)
+		(start 106.416765 79.483235)
+		(end 106.133921 79.483235)
 		(width 0.2)
 		(layer "F.Cu")
@@
 	)
 	(segment
-		(start 97.43 73.935)
-		(end 96.67 74.695)
+		(start 109.115 85.08)
+		(end 110.614455 85.08)
+		(width 0.2)
+		(layer "F.Cu")
+		(net 87)
+	)
+	(segment
+		(start 100.585686 73.935)
+		(end 96.16 73.935)
 		(width 0.2)
 		(layer "F.Cu")
