File: atslim-328.kicad_sch (KiCad schematic)
At the start: 13 parts, among them J1 UPDI, J2 RESET, J6 GPIO, U1 ATmega3208-M

Commit message: Recent updates
Connections:
- net +3V3: now also J6.1 (Pin_1); no longer J6.2 (Pin_2)
- net GND: now also J6.2 (Pin_2); no longer J6.1 (Pin_1)
Changed lines of the file:
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@@
-	(wire
-		(pts
-			(xy 261.62 30.48) (xy 273.05 30.48)
-		)
-		(stroke
-			(width 0)
-			(type default)
-		)
-	)
 	(wire
 		(pts
@@
 		(pts
 			(xy 203.2 109.22) (xy 214.63 109.22)
+		)
+		(stroke
+			(width 0)
+			(type default)
+		)
+	)
+	(wire
+		(pts
+			(xy 248.92 30.48) (xy 237.49 30.48)
 		)
 		(stroke
@@
 		)
 	)
-	(global_label "+3V3"
-		(shape input)
-		(at 273.05 30.48 0)
-		(fields_autoplaced yes)
-		(effects
-			(font
-				(size 1.27 1.27)
-			)
-			(justify left)
-		)
-		(property "Intersheetrefs" "${INTERSHEET_REFS}"
-			(at 281.1152 30.48 0)
-			(effects
-				(font
-					(size 1.27 1.27)
-				)
-				(justify left)
-				(hide yes)
-			)
-		)
-	)
 	(global_label "RESET"
 		(shape output)
@@
 				)
 				(justify left)
+				(hide yes)
+			)
+		)
+	)
+	(global_label "+3V3"
+		(shape input)
+		(at 237.49 30.48 180)
+		(fields_autoplaced yes)
+		(effects
+			(font
+				(size 1.27 1.27)
+			)
+			(justify right)
+		)
+		(property "Intersheetrefs" "${INTERSHEET_REFS}"
+			(at 229.4248 30.48 0)
+			(effects
+				(font
+					(size 1.27 1.27)
+				)
+				(justify right)
 				(hide yes)
 			)
@@
 	(symbol
 		(lib_id "power:GND")
-		(at 248.92 30.48 270)
+		(at 261.62 30.48 90)
 		(unit 1)
 		(exclude_from_sim no)
@@
 		(dnp no)
 		(property "Reference" "#PWR022"
-			(at 242.57 30.48 0)
+			(at 267.97 30.48 0)
 			(effects
 				(font
@@
 		)
 		(property "Value" "GND"
-			(at 247.396 27.686 90)
+			(at 264.16 29.21 90)
 			(effects
 				(font
@@
 		)
 		(property "Footprint" ""
-			(at 248.92 30.48 0)
+			(at 261.62 30.48 0)
 			(effects
 				(font
@@
 		)
 		(property "Datasheet" ""
-			(at 248.92 30.48 0)
+			(at 261.62 30.48 0)
 			(effects
 				(font
@@
 		)
 		(property "Description" "Power symbol creates a global label with name \"GND\" , ground"
-			(at 248.92 30.48 0)
-			(effects
-				(font
+			(at 261.62 30.48 0)
+			(effects
+				(font

Commit message: Fucked up UPDI... of course
Connections:
- net Prog_TX: now also J1.5 (TX); no longer J1.3 (TX)
Changed lines of the file:
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@@
+	)
+	(no_connect
+		(at 87.63 88.9)
 	)
 	(no_connect
@@
 	)
 	(no_connect
-		(at 87.63 83.82)
-	)
-	(no_connect
 		(at 149.86 133.35)
 	)
@@
 	(wire
 		(pts
+			(xy 87.63 83.82) (xy 95.25 83.82)
+		)
+		(stroke
+			(width 0)
+			(type default)
+		)
+	)
+	(wire
+		(pts
 			(xy 237.49 53.34) (xy 248.92 53.34)
 		)
@@
 		(pts
 			(xy 237.49 45.72) (xy 248.92 45.72)
-		)
-		(stroke
-			(width 0)
-			(type default)
-		)
-	)
-	(wire
-		(pts
-			(xy 87.63 88.9) (xy 95.25 88.9)
 		)
 		(stroke
@@
 		)
 	)
-	(global_label "+5V"
+	(global_label "Prog_TX"
 		(shape input)
-		(at 77.47 74.93 90)
+		(at 95.25 83.82 0)
 		(fields_autoplaced yes)
 		(effects
@@
 		)
 		(property "Intersheetrefs" "${INTERSHEET_REFS}"
-			(at 77.47 68.0743 90)
+			(at 106.0366 83.82 0)
 			(effects
 				(font
@@
 		)
 	)
-	(global_label "Prog_TX"
+	(global_label "+5V"
 		(shape input)
-		(at 95.25 88.9 0)
+		(at 77.47 74.93 90)
 		(fields_autoplaced yes)
 		(effects
@@
 		)
 		(property "Intersheetrefs" "${INTERSHEET_REFS}"
-			(at 106.0366 88.9 0)
+			(at 77.47 68.0743 90)
 			(effects
 				(font
